Commit message: v0.3.9 -  add a gui controller, fixing bugs in the hand

File: robot_arm_description/urdf/robot_arm.urdf (robot description, URDF)
Before this commit: robot robot_arm, 10 links, 9 joints
Joints:
- joint finger_1_joint: limit lower=-1.2217 upper=0.0 effort=2.0 velocity=2.0 -> lower=0.0 upper=1.2217 effort=2.0 velocity=2.0
- joint finger_2_joint: axis 0.866 0.5 0 -> 0 1 0; limit lower=-1.2217 upper=0.0 effort=2.0 velocity=2.0 -> lower=0.0 upper=1.2217 effort=2.0 velocity=2.0
- joint finger_3_joint: axis 0.866 -0.5 0 -> 0 1 0; limit lower=-1.2217 upper=0.0 effort=2.0 velocity=2.0 -> lower=0.0 upper=1.2217 effort=2.0 velocity=2.0
- joint shoulder_roll: axis 1 0 0 -> 0 1 0

Commit message: fixed gripper movement

File: robot_arm_description/urdf/robot_arm.urdf (robot description, URDF)
Before this commit: robot robot_arm, 10 links, 9 joints
Joints:
- joint finger_1_joint: limit lower=0.0 upper=1.2217 effort=2.0 velocity=2.0 -> lower=-1.2217 upper=0.0 effort=2.0 velocity=2.0
- joint finger_2_joint: limit lower=0.0 upper=1.2217 effort=2.0 velocity=2.0 -> lower=-1.2217 upper=0.0 effort=2.0 velocity=2.0
- joint finger_3_joint: limit lower=0.0 upper=1.2217 effort=2.0 velocity=2.0 -> lower=-1.2217 upper=0.0 effort=2.0 velocity=2.0

Commit message: v0.4.2 - got camera working

File: robot_arm_description/urdf/robot_arm.urdf (robot description, URDF)
Before this commit: robot robot_arm, 10 links, 9 joints
Links:
- added link camera_link, mass 0.05; collision box size=0.04 0.04 0.02; visual box size=0.04 0.04 0.02
Joints:
- added joint camera_joint: type fixed, parent wrist_link, child camera_link, origin xyz=0.03 0 0.02 rpy=0 0 0

Commit message: v0.4.4 - working chess GUI, bug fixes

File: robot_arm_description/urdf/robot_arm.urdf (robot description, URDF)
Before this commit: robot robot_arm, 11 links, 10 joints
Joints:
- joint camera_joint: origin xyz=0.03 0 0.02 rpy=0 0 0 -> xyz=0 0 0.04 rpy=0 1.5708 0

Commit message: v0.4.5 - bug fixes -right standby postion- Wokring ON board detection

File: robot_arm_description/urdf/robot_arm.urdf (robot description, URDF)
Before this commit: robot robot_arm, 11 links, 10 joints
Joints:
- joint camera_joint: origin xyz=0 0 0.04 rpy=0 1.5708 0 -> xyz=0.04 0 0.02 rpy=0 0 0
